Commit message: Modify lwa4 to crichton specification?

File: schunk_description/urdf/lwa4d/lwa4d.urdf.xacro (robot description, xacro)
@@ -108,14 +108,14 @@
 -->
       <visual>
-        <origin xyz="0 0 -0.39" rpy="0 0 ${M_PI}"/>
-        <geometry>
-          <mesh filename="package://schunk_description/meshes/lwa4d/arm_3_link.stl"/>
-        </geometry>
-        <material name="Schunk/LightGrey"/>
-      </visual>
-      <collision>
-        <origin xyz="0 0 -0.39" rpy="0 0 ${M_PI}"/>
-        <geometry>
-          <mesh filename="package://schunk_description/meshes/lwa4d/arm_3_link_collision.stl"/>
+        <origin xyz="0 0 -0.328" rpy="0 0 ${M_PI}"/>
+        <geometry>
+          <mesh filename="package://schunk_description/meshes/lwa4d/arm_3_link_shortened.stl"/>
+        </geometry>
+        <material name="Schunk/LightGrey"/>
+      </visual>
+      <collision>
+        <origin xyz="0 0 -0.328" rpy="0 0 ${M_PI}"/>
+        <geometry>
+          <mesh filename="package://schunk_description/meshes/lwa4d/arm_3_link_shortened_collision.stl"/>
         </geometry>
       </collision>
@@ -123,5 +123,5 @@
     <!-- joint between arm_3_link and arm_4_link -->
     <joint name="${name}_4_joint" type="revolute">
-      <origin xyz="0 0 -0.39" rpy="-${M_PI/2} 0 0"/>
+      <origin xyz="0 0 -0.328" rpy="-${M_PI/2} 0 0"/>
       <parent link="${name}_3_link"/>
       <child link="${name}_4_link"/>

File: schunk_description/urdf/materials.urdf.xacro (robot description, xacro)
@@ -8,5 +8,5 @@
   </material>
   <material name="Schunk/Black">
-    <color rgba="0.0 0.0 0.0 1.0"/>
+    <color rgba="0.05 0.05 0.05 1.0"/>
   </material>
   <material name="Schunk/DarkGolden">
